File: wifi.sch (KiCad schematic (older format))
At the start: 130 parts, among them J1 Conn_02x10_Odd_Even, J11 Conn_Coaxial, J12 Conn_02x05_Counter_Clockwise, J13 Conn_02x03_Odd_Even, J14 Conn_01x02, J15 Conn_01x02, J16 Conn_01x02, J2 Conn_02x10_Odd_Even, J21 Conn_02x04_Odd_Even, J22 Conn_01x03, J23 Conn_01x03, J24 Conn_01x02, J3 Conn_02x06_Odd_Even, J5 Conn_01x03, J6 Conn_01x03, J7 Conn_02x07_Odd_Even, J9 Conn_01x02, Q2 TP0610T, Q3 BSS138, Q4 BSS138, Q5 BSS138, SW2 SW_DIP_x01, SW3 SW_DIP_x01, U1 CC3220SM2ARGKT, U10 TMP100, U8 MX25R3235FM1IL0, U9 OPA4340UA, Y2 32.768kHz, Y3 Crystal_GND24_Small

Commit message: Fixes for Aisler
Parts:
- added FID1, FID2, FID3: Fiducial, Fiducial:Fiducial_0.5mm_Mask1mm, symbol Mechanical:Fiducial
- added R45, R75, R78, R81, R85, R89, R91: 0, Resistor_SMD:R_0402_1005Metric, symbol Device:R_Small
- AE1: MFG Name (none) -> Taiyo Yuden; MFG Part Num (none) -> AH316M245001-T
- C27: MFG Name (none) -> Murata; MFG Part Num (none) -> GRM155R61A105KE15D
- C28, C32, C33, C36, C37, C38, C43, C44, C46, C47, C57: MFG Name (none) -> TDK; MFG Part Num (none) -> C1005X5R1A104K050BA
- C29, C30, C31: MFG Name (none) -> TDK; MFG Part Num (none) -> C1005X5R0J475M050BC
- C34: MFG Name (none) -> Murata; MFG Part Num (none) -> GJM1555C1HR50BB01J
- C35: footprint Capacitor_SMD:C_0402_1005Metric -> Capacitor_SMD:C_0603_1608Metric; MFG Name (none) -> Murata; MFG Part Num (none) -> GRM188R60J106ME47D
- C45: MFG Name (none) -> Murata; MFG Part Num (none) -> GRM188R60J106ME47D
- C48, C49: MFG Name (none) -> Murata; MFG Part Num (none) -> GRM1555C1H100JA01D
- C50, C51: MFG Name (none) -> Murata; MFG Part Num (none) -> GRM1555C1H6R2CA01D
- C52: MFG Name (none) -> Murata; MFG Part Num (none) -> GRM155R61A103KA01D
- C53, C54, C55, C56: MFG Name (none) -> TDK; MFG Part Num (none) -> C1005X7R1C103K
- D10: MFG Name (none) -> Rohm; MFG Part Num (none) -> SML-311UTT86
- D4, D5: MFG Name (none) -> Bourns; MFG Part Num (none) -> CD0603-B00340
- D8: MFG Name (none) -> Lumex; MFG Part Num (none) -> SML-LX0603GW-TR
- D9: MFG Name (none) -> Wurth Elektronik eiSos; MFG Part Num (none) -> 150060YS75000
- FL1: MFG Name (none) -> TDK; MFG Part Num (none) -> DEA202450BT-1294C1-H
- J11: MFG Name (none) -> Murata; MFG Part Num (none) -> MM8030-2610RJ3
- J13: MFG Name (none) -> Wurth Elektronik; MFG Part Num (none) -> '61300621121
- J14, J15, J16, J21, J24, J9: MFG Name (none) -> Wurth Elektronik; MFG Part Num (none) -> '61300211121
- J22, J23, J5, J6: MFG Name (none) -> Wurth Elektronik; MFG Part Num (none) -> '61300311121
- J3: MFG Name (none) -> Wurth Elektronik; MFG Part Num (none) -> '61301021121
- J7: MFG Name (none) -> Samtec; MFG Part Num (none) -> FTSH-107-01-F-DV
- L3: MFG Name (none) -> Murata; MFG Part Num (none) -> LQG15HS3N3S02D
- L4, L6: MFG Name (none) -> Murata; MFG Part Num (none) -> LQM2HPN2R2MG0L
- L5: MFG Name (none) -> Murata; MFG Part Num (none) -> LQM2HPN1R0MG0L
- Q2: MFG Name (none) -> Diodes Inc; MFG Part Num (none) -> BSS84DW-7-F
- Q3, Q5: MFG Name (none) -> Fairchild; MFG Part Num (none) -> FDN358P
- Q4: MFG Name (none) -> Fairchild; MFG Part Num (none) -> BSS138
- R102, R105, R110, R111: MFG Name (none) -> Panasonic; MFG Part Num (none) -> ERJ-2RKF4700X
- R103, R104, R112, R113: MFG Name (none) -> Vishay-Dale; MFG Part Num (none) -> CRCW0402576KFKED
- R106, R107, R114, R115: MFG Name (none) -> Vishay-Dale; MFG Part Num (none) -> CRCW0402422KFKED
- R116, R123, R128, R129, R134, R135, R154, R39, R40, R43, R44, R67, R68, R71, R72, R76, R80, R82, R84, R86, R87, R88, R90, R92: MFG Name (none) -> Panasonic; MFG Part Num (none) -> ERJ-2GE0R00X
- R118, R119: MFG Name (none) -> Vishay-Dale; MFG Part Num (none) -> CRCW04023K30JNED
- R136, R151, R152, R153, R41, R49, R50: MFG Name (none) -> Vishay-Dale; MFG Part Num (none) -> CRCW0402100KJNED
- R138, R139, R30: MFG Name (none) -> Vishay-Dale; MFG Part Num (none) -> CRCW04021K00JNED
- R141, R142, R35, R53: MFG Name (none) -> Vishay-Dale; MFG Part Num (none) -> CRCW040210K0JNED
- R147, R148, R149: MFG Name (none) -> Vishay-Dale; MFG Part Num (none) -> CRCW0603270RJNEA
- R33, R34: MFG Name (none) -> Vishay-Dale; MFG Part Num (none) -> CRCW060333R0JNEA
- R36, R57: MFG Name (none) -> Panasonic; MFG Part Num (none) -> ERJ-3GEY0R00V
- R47: MFG Name (none) -> Vishay-Dale; MFG Part Num (none) -> CRCW0402270RJNED
- R51: MFG Name (none) -> Vishay-Dale; MFG Part Num (none) -> CRCW04022K70JNED
- R52: MFG Name (none) -> Vishay-Dale; MFG Part Num (none) -> CRCW04022K20JNED
- SW2, SW3: MFG Name (none) -> APEM; MFG Part Num (none) -> MJTP1117
- U1: footprint Package_DFN_QFN:Texas_S-PVQFN-N64_EP4.25x4.25mm -> Package_DFN_QFN:Texas_S-PVQFN-N64_EP4.25x4.25mm_ThermalVias
- U10: MFG Name (none) -> Texas Instruments; MFG Part Num (none) -> TMP100
- U8: MFG Name (none) -> Macronix; MFG Part Num (none) -> MX25R3235FM1IL0
- U9: MFG Name (none) -> Texas Instruments; MFG Part Num (none) -> OPA4342EA/250
- Y2: MFG Name (none) -> Abracon; MFG Part Num (none) -> ABS07-32.768KHZ-9-T
- Y3: MFG Name (none) -> Epson; MFG Part Num (none) -> Q24FA20H0039600
Connections:
- net GND: now also J2.2 (Pin_2)
- net P01_GPIO_10: now also R89.2
- net P02_GPIO_11: now also R91.2
- net P21_GPIO_25: now also R78.1
- net P61_GPIO_06: now also R75.2
- net P20_JTAG_TMS: now reaches J3.10 (Pin_10)
- net P20_JTAG_TMS: now also U1.20 (TMS)
- net P17_GPIO_24: now reaches J3.4 (Pin_4)
- net P17_GPIO_24: now also U1.17 (TDO), R85.2
- net P16_JTAG_TDI: now reaches J3.6 (Pin_6)
- net P16_JTAG_TDI: now also U1.16 (TDI), R45.2
- net P19_JTAG_TCK: now reaches J3.8 (Pin_8)
- net P19_JTAG_TCK: now also U1.19 (TCK)
- net P18_GPIO_28: now reaches U1.18 (GPIO28)
- net at J1.17 (Pin_17): now also R89.1
- net at J1.19 (Pin_19): now also R91.1
- net at J1.9 (Pin_9): now also R75.1
- net at J2.16 (Pin_16): now also R78.2
- net at J2.17 (Pin_17): now also R81.1
- net at J2.19 (Pin_19): now also R85.1
- new net P16_GPIO_23: R45.1, R81.2

Commit message: MODASF initial commit
Parts:
- removed AE1: Antenna_Chip, pwrcon:Taiyo_WLAN, symbol Device:Antenna_Chip
- removed C27: 1uF, Capacitor_SMD:C_0402_1005Metric, symbol Device:C_Small
- removed C28, C32, C33, C37, C38, C43, C44, C46, C47: 0.1uF, Capacitor_SMD:C_0402_1005Metric, symbol Device:C_Small
- removed C29: 4.7uF, Capacitor_SMD:C_0402_1005Metric, symbol Device:C_Small
- removed C34: 0.5pF, Capacitor_SMD:C_0402_1005Metric, symbol Device:C_Small
- removed C35, C45: 10uF, Capacitor_SMD:C_0603_1608Metric, symbol Device:C_Small
- removed C36: 10uF, Capacitor_SMD:C_0402_1005Metric, symbol Device:C_Small
- removed C48, C49, C50, C51: 6.2pF, Capacitor_SMD:C_0402_1005Metric, symbol Device:C_Small
- removed FL1: BFCN-2450, pwrcon:TDK_Filter, symbol RF_Filter:BFCN-2450
- removed J11: Conn_Coaxial, pwrcon:Co-axial_Connector_RF, symbol Connector:Conn_Coaxial
- removed J14: Conn_01x02, Connector_PinHeader_2.54mm:PinHeader_1x02_P2.54mm_Vertical, symbol Connector_Generic:Conn_01x02
- removed J21: Conn_02x04_Odd_Even, Connector_PinSocket_2.54mm:PinSocket_2x04_P2.54mm_Vertical, symbol Connector_Generic:Conn_02x04_Odd_Even
- removed L3: L_Core_Ferrite_Small, Inductor_SMD:L_01005_0402Metric, symbol Device:L_Core_Ferrite_Small
- removed L4, L6: 2.2uH, Inductor_SMD:L_Wuerth_MAPI-2512, symbol Device:L_Core_Ferrite_Small
- removed L5: 1uH, Inductor_SMD:L_Wuerth_MAPI-2512, symbol Device:L_Core_Ferrite_Small
- removed R128, R39, R40, R43: 0, Resistor_SMD:R_0402_1005Metric, symbol Device:R_Small
- removed R35: 10K, Resistor_SMD:R_0402_1005Metric, symbol Device:R_Small
- removed R36: 0, Resistor_SMD:R_0603_1608Metric, symbol Device:R_Small
- removed R41: 10k, Resistor_SMD:R_0402_1005Metric, symbol Device:R_Small
- removed R49, R50: 100K, Resistor_SMD:R_0402_1005Metric, symbol Device:R_Small
- removed R51: 2.7K, Resistor_SMD:R_0402_1005Metric, symbol Device:R_Small
- removed U1: CC3220SM2ARGKT, Package_DFN_QFN:Texas_S-PVQFN-N64_EP4.25x4.25mm_ThermalVias, symbol MCU_TI:CC3220SM2ARGKT
- removed U10: TMP100, Package_TO_SOT_SMD:SOT-23-6, symbol Sensor_Temperature:TMP100
- removed U8: MX25R3235FM1IL0, Package_SO:SOIC-8_3.9x4.9mm_P1.27mm, symbol Memory_Flash:W25Q32JVSS
- removed Y2: 32.768kHz, Crystal:Crystal_SMD_3215-2Pin_3.2x1.5mm, symbol Device:Crystal_Small
- removed Y3: Crystal_GND24_Small, Crystal:Crystal_SMD_2520-4Pin_2.5x2.0mm, symbol Device:Crystal_GND24_Small
- added C41: 100uF, Capacitor_SMD:C_0402_1005Metric, symbol Device:C_Small
- added J10, J16, J17, J18, J19, J20: Conn_01x02, Connector_PinHeader_2.54mm:PinHeader_1x02_P2.54mm_Vertical, symbol Connector_Generic:Conn_01x02
- added J22: Conn_01x03, Connector_PinHeader_2.54mm:PinHeader_1x03_P2.54mm_Vertical, symbol Connector_Generic:Conn_01x03
- added R104, R42, R46, R52, R56, R65: 0, Resistor_SMD:R_0402_1005Metric, symbol Device:R_Small
- added TP1: TestPoint, TestPoint:TestPoint_Pad_D2.0mm, symbol Connector:TestPoint
- added U1: CC3220MODASF12MONR, TIMOD_footprints:CC3220MODASF12MONR, symbol wifi-rescue:CC3220MODASF12MONR-2020-05-13_17-39-37
- added U10: TMP006AIYZFR, TMP006_footprints:TMP006AIYZFR, symbol TMP006AIYZFR:TMP006AIYZFR
- C33: renamed from C30; value 4.7uF -> 0.1uF
- C34: renamed from C31; value 4.7uF -> 0.1uF
- C42: value 10uF -> 100uF; footprint Capacitor_SMD:C_0603_1608Metric -> Capacitor_SMD:C_0402_1005Metric; MFG Name (none) -> TDK; MFG Part Num (none) -> C1005X5R0J475M050BC
- Q5: renamed from Q2; MFG Part Num BSS84DW-7-F -> FDN358P
- R119: value 3.3K -> 0
- R126: renamed from R118; value 3.3K -> 0
- R145: renamed from R147; value 270 -> 750
- R146: renamed from R148; value 270 -> 750
- R147: renamed from R149; value 270 -> 750
- renumbered C52 to C26, C53 to C27, C54 to C28, C55 to C29, C56 to C30, C57 to C35, D8 to D7, J12 to J112, J13 to J12, J15 to J14, J16 to J15, J22 to J21, J23 to J26, Q3 to Q4, Q4 to Q6, Q5 to Q7, R45 to R105, R47 to R107, R52 to R109, R53 to R113, R116 to R114, R123 to R121, R129 to R127, R134 to R132, R135 to R133, R136 to R134, R138 to R136, R139 to R137, R141 to R139, R142 to R140, R151 to R149, R152 to R150, R153 to R151, R154 to R152, R30 to R31, R57 to R38, R67 to R49, R68 to R50, R71 to R53, R72 to R54, R75 to R57, R76 to R58, R78 to R60, R80 to R62, R81 to R63, R82 to R64, R84 to R66, R85 to R67, R86 to R68, R87 to R69, R88 to R70, R89 to R71, R90 to R72, R91 to R73, R92 to R74, R102 to R84, R103 to R85, R104 to R86, R105 to R87, R106 to R88, R107 to R89, R110 to R92, R111 to R93, R112 to R94, R113 to R95, R114 to R96, R115 to R97
Connections:
- net VDD_DIG_CC is gone; now on net VBAT_CC: C42.2
- net GND: now also R126.1, C41.1, J20.1 (Pin_1), J20.2 (Pin_2), J22.2 (Pin_2), J22.3 (Pin_3), U1.1 (GND), U1.16 (GND), U1.2 (GND), U1.27 (GND), U1.28 (GND), U1.30 (GND), U1.32 (GND), U1.38 (GND), U1.43 (GND), U1.55 (GND), U1.56 (GND), U1.57 (GND), U1.58 (GND), U1.59 (GND), U1.60 (GND), U1.61 (GND), U1.62 (GND), U1.63 (GND), U10.A1 (DGND), U10.A2 (AGND); no longer J26.2 (Pin_2), J26.3 (Pin_3), R44.2
- net P01_GPIO_10: now also U1.3 (GPIO_10)
- net P02_GPIO_11: now also U1.4 (GPIO_11)
- net P03_GPIO_12: now also U1.9 (GPIO_12)
- net P04_GPIO_13: now also U1.10 (GPIO_13)
- net P05_GPIO_14: now also R65.2, U1.5 (GPIO_14)
- net P06_GPIO_15: now also R56.1, U1.6 (GPIO_15)
- net P07_GPIO_16: now also R52.1, U1.7 (GPIO_16)
- net P08_GPIO_17: now also R44.1, U1.8 (GPIO_17)
- net P15_GPIO_22: now also U1.11 (GPIO_22)
- net P16_GPIO_23: now also R105.2; no longer R105.1
- net P16_JTAG_TDI: now also R105.1, U1.12 (JTAG_TDI); no longer R105.2
- net P17_GPIO_24: now also R104.2; no longer J3.4 (Pin_4)
- net P18_GPIO_28: now also R42.1, U1.19 (GPIO_28)
- net P19_JTAG_TCK: now also U1.21 (JTAG_TCK)
- net P20_JTAG_TMS: now also U1.22 (JTAG_TMS)
- net P50_GPIO_00: now also U1.44 (GPIO_0)
- net P53_GPIO_30: now also U1.42 (GPIO_30)
- net P55_GPIO_01: now also U1.46 (GPIO_01)
- net P57_GPIO_02: now also U1.47 (GPIO_02)
- net P58_GPIO_03: now also U1.48 (GPIO_03)
- net P59_GPIO_04: now also U1.49 (GPIO_04)
- net P60_GPIO_05: now also U1.50 (GPIO_05)
- net P61_GPIO_06: now also U1.51 (GPIO_06)
- net P62_GPIO_07: now also U1.52 (GPIO_07)
- net P63_GPIO_08: now also U1.53 (GPIO_08)
- net P64_GPIO_09: now also U1.54 (GPIO_09)
- net SENS_I2C_SCL: now also U10.C3 (SDA); no longer R119.2, R132.2
- net SENS_I2C_SDA: now also U10.B3 (SCL); no longer R126.1, R133.2
- net SOP0: now also U1.34 (SOP0)
- net SOP1: now also U1.24 (SOP1)
- net SOP2: now also U1.23 (SOP2)
- net VBAT_CC: now also J26.3 (Pin_3), R38.2, C41.2, J10.2 (Pin_2), J18.2 (Pin_2), U1.37 (VBAT1), U1.40 (VBAT2); no longer J9.2 (Pin_2)
- net VCC_5V: now also J19.2 (Pin_2), J22.1 (Pin_1); no longer J26.1 (Pin_1)
- net VCC_BRD: now also J26.1 (Pin_1), J9.1 (Pin_1), R119.2, J16.2 (Pin_2), J17.1 (Pin_1); no longer R107.1, R114.1, R119.1, R126.2, R38.1
- net VCC_OPAMP: now also J9.2 (Pin_2)
- net at J7.1 (Pin_1), J7.2 (Pin_2): now also TP1.1
- net at J12.1 (Pin_1), J12.3 (Pin_3), J12.5 (Pin_5): now also R107.1; no longer R107.2
- net at C35.2, R114.2: now also U10.A3 (V+)
- net PWR: now reaches J1.1 (Pin_1)
- net PWR: now also R38.1; no longer R38.2
- net RX: now reaches J1.5 (Pin_5), R49.1
- net TX: now reaches J1.7 (Pin_7), R53.1
- net at J1.13 (Pin_13): now also R65.1
- net GPIO: now reaches J1.9 (Pin_9), R57.1
- net at J2.12 (Pin_12): now also R52.2
- net at J2.14 (Pin_14): now also R56.2
- net at J2.4 (Pin_4): now also R42.2
- net at J2.6 (Pin_6): now also R44.2
- net at J2.8 (Pin_8): now also R46.2
- new net: J26.2 (Pin_2), R107.2
- new net: R119.1, U10.C1 (SDR0)
- new net: R126.2, U10.B1 (ADR1)
- new net: J10.1 (Pin_1), U1.36 (VBAT_RESET)
- new net P17_JTAG_TDO: J3.4 (Pin_4), R104.1, U1.18 (JTAG_TDO)
- new net P29_GPIO_26: U1.25 (ANT_SEL1)
- new net P30_GPIO_27: U1.26 (ANT_SEL2)
- new net P45_GPIO_31: R46.1
- new net SPI_CLK: U1.15 (FLASH_SPI_CLK)
- new net SPI_CS_IN: U1.14 (FLASH_SPI_CS_IN_N)
- new net SPI_MISO: U1.13 (FLASH_SPI_MISO)
- new net SPI_MOSI: U1.17 (FLASH_SPI_MOSI)
- new net VBUS_USB1: J19.1 (Pin_1)
- new net VCC_Buffer: J17.2 (Pin_2)
- new net VCC_LDO_3V3: J16.1 (Pin_1), J18.1 (Pin_1)
Other:
- note added: "GPIO"
- note added: "RESET"
- note added: "SPI_CS"
- note added: "SPI_MISO"
- note added: "SPI_MOSI"
- note added: "TEST"
- moved on the sheet: C26, C27, C28, C29, C30, C33, C34, C35, FID3, J1, J112, J14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

Commit message: Updated BoM, decided to use 3 LEDs and switches from cc3220s layout
Parts:
- C33, C34: MFG Name TDK -> Murata; MFG Part Num C1005X5R0J475M050BC -> GRM155R61A104KA01D
- C35: MFG Name TDK -> Murata; MFG Part Num C1005X5R1A104K050BA -> GRM155R61A104KA01D
- C41, C42: MFG Name TDK -> Murata; MFG Part Num C1005X5R0J475M050BC -> GRM31CR60J107ME39L
- J2: MFG Name (none) -> Wurth; MFG Part Num (none) -> '61300311121
- Q4, Q7: MFG Part Num FDN358P -> BSS138
- R119, R126: MFG Name Vishay-Dale -> Panasonic; MFG Part Num CRCW04023K30JNED -> ERJ-2GE0R00X
- R145, R146, R147: value 750 -> 270
- U10: MFG Name (none) -> TI; MFG Part Num (none) -> TMP006AIYZF
- U9: renamed from U1; MFG Name (none) -> TI; MFG Part Num (none) -> CC3220MODASF12MONR
- renumbered D7 to D8, U9 to U7
Connections:
- net SENS_I2C_SCL: now also R132.2; no longer U10.C3 (SDA)
- net SENS_I2C_SDA: now also R133.1; no longer U10.B3 (SCL)
- net VCC_BRD: now also R114.1
- net at R132.1: now also U10.B3 (SCL)
- net at R133.2: now also U10.C3 (SDA)
Other:
- moved on the sheet: R132, R133
Changed lines of the file:
@@
 $EndDescr
 $Comp
-L Amplifier_Operational:OPA4340UA U9
+L Amplifier_Operational:OPA4340UA U7
 U 1 1 5E321612
 P 8075 4150
-F 0 "U9" H 8075 4517 50  0000 C CNN
+F 0 "U7" H 8075 4517 50  0000 C CNN
 F 1 "OPA4340UA" H 8075 4426 50  0000 C CNN
 F 2 "Package_SO:TSSOP-14_4.4x5mm_P0.65mm" H 8025 4250 50  0001 C CNN
@@
 $EndComp
 $Comp
-L Amplifier_Operational:OPA4340UA U9
+L Amplifier_Operational:OPA4340UA U7
 U 2 1 5E32274A
 P 8125 4800
-F 0 "U9" H 8125 5167 50  0000 C CNN
+F 0 "U7" H 8125 5167 50  0000 C CNN
 F 1 "OPA4340UA" H 8125 5076 50  0000 C CNN
 F 2 "Package_SO:TSSOP-14_4.4x5mm_P0.65mm" H 8075 4900 50  0001 C CNN
@@
 $EndComp
 $Comp
-L Amplifier_Operational:OPA4340UA U9
+L Amplifier_Operational:OPA4340UA U7
 U 3 1 5E324323
 P 9400 4075
-F 0 "U9" H 9400 4442 50  0000 C CNN
+F 0 "U7" H 9400 4442 50  0000 C CNN
 F 1 "OPA4340UA" H 9400 4351 50  0000 C CNN
 F 2 "Package_SO:TSSOP-14_4.4x5mm_P0.65mm" H 9350 4175 50  0001 C CNN
@@
 $EndComp
 $Comp
-L Amplifier_Operational:OPA4340UA U9
+L Amplifier_Operational:OPA4340UA U7
 U 4 1 5E3260D2
 P 9450 4825
-F 0 "U9" H 9450 5192 50  0000 C CNN
+F 0 "U7" H 9450 5192 50  0000 C CNN
 F 1 "OPA4340UA" H 9450 5101 50  0000 C CNN
 F 2 "Package_SO:TSSOP-14_4.4x5mm_P0.65mm" H 9400 4925 50  0001 C CNN
@@
 	9700 4275 9700 4075
 $Comp
-L Amplifier_Operational:OPA4340UA U9
+L Amplifier_Operational:OPA4340UA U7
 U 5 1 5DB6D511
 P 10625 4475
-F 0 "U9" H 10583 4521 50  0000 L CNN
+F 0 "U7" H 10583 4521 50  0000 L CNN
 F 1 "OPA4340UA" H 10583 4430 50  0000 L CNN
 F 2 "Package_SO:TSSOP-14_4.4x5mm_P0.65mm" H 10575 4575 50  0001 C CNN
@@
 F 2 "Capacitor_SMD:C_0402_1005Metric" H 3600 2625 50  0001 C CNN
 F 3 "~" H 3600 2625 50  0001 C CNN
-F 4 "TDK" H 3600 2625 50  0001 C CNN "MFG Name"
-F 5 "C1005X5R0J475M050BC" H 3600 2625 50  0001 C CNN "MFG Part Num"
+F 4 "Murata" H 3600 2625 50  0001 C CNN "MFG Name"
+F 5 "GRM155R61A104KA01D" H 3600 2625 50  0001 C CNN "MFG Part Num"
 	1    3600 2625
 	0    1    1    0
@@
 F 2 "Capacitor_SMD:C_0402_1005Metric" H 3275 2625 50  0001 C CNN
 F 3 "~" H 3275 2625 50  0001 C CNN
-F 4 "TDK" H 3275 2625 50  0001 C CNN "MFG Name"
-F 5 "C1005X5R0J475M050BC" H 3275 2625 50  0001 C CNN "MFG Part Num"
+F 4 "Murata" H 3275 2625 50  0001 C CNN "MFG Name"
+F 5 "GRM155R61A104KA01D" H 3275 2625 50  0001 C CNN "MFG Part Num"
 	1    3275 2625
 	0    1    1    0
@@
 U 1 1 5DCB12DD
 P 7650 6100
-F 0 "R152" V 7846 6100 50  0001 C CNN
+F 0 "R152" V 7846 6100 50  0000 C CNN
 F 1 "0" V 7755 6100 50  0001 C CNN
 F 2 "Resistor_SMD:R_0402_1005Metric" H 7650 6100 50  0001 C CNN
@@
 	7450 5925 7450 5700
 $Comp
-L Device:LED D7
+L Device:LED D8
 U 1 1 5DCCC072
 P 8875 5550
-F 0 "D7" V 8868 5433 50  0000 R CNN
+F 0 "D8" V 8868 5433 50  0000 R CNN
 F 1 "LED" H 8868 5675 50  0001 C CNN
 F 2 "LED_SMD:LED_0603_1608Metric" H 8875 5550 50  0001 C CNN
@@
 F 3 "http://www.diodes.com/assets/Datasheets/ds31898.pdf" H 8775 6100 50  0001 L CNN
 F 4 "Fairchild" H 8775 6100 50  0001 C CNN "MFG Name"
-F 5 "FDN358P" H 8775 6100 50  0001 C CNN "MFG Part Num"
+F 5 "BSS138" H 8775 6100 50  0001 C CNN "MFG Part Num"
 	1    8775 6100
 	1    0    0    -1
@@
 F 3 "http://www.diodes.com/assets/Datasheets/ds31898.pdf" H 9900 6100 50  0001 L CNN
 F 4 "Fairchild" H 9900 6100 50  0001 C CNN "MFG Name"
-F 5 "FDN358P" H 9900 6100 50  0001 C CNN "MFG Part Num"
+F 5 "BSS138" H 9900 6100 50  0001 C CNN "MFG Part Num"
 	1    9900 6100
 	1    0    0    -1
@@
 P 8875 5800
 F 0 "R146" V 8950 5800 50  0000 C CNN
-F 1 "750" V 8800 5800 50  0000 C CNN
+F 1 "270" V 8800 5800 50  0000 C CNN
 F 2 "Resistor_SMD:R_0603_1608Metric" H 8875 5800 50  0001 C CNN
 F 3 "~" H 8875 5800 50  0001 C CNN
@@
 P 9475 5800
 F 0 "R145" V 9550 5800 50  0000 C CNN
-F 1 "750" V 9400 5800 50  0000 C CNN
+F 1 "270" V 9400 5800 50  0000 C CNN
 F 2 "Resistor_SMD:R_0603_1608Metric" H 9475 5800 50  0001 C CNN
 F 3 "~" H 9475 5800 50  0001 C CNN
@@
 P 10000 5800
 F 0 "R147" V 10075 5800 50  0000 C CNN
-F 1 "750" V 9925 5800 50  0000 C CNN
+F 1 "270" V 9925 5800 50  0000 C CNN
 F 2 "Resistor_SMD:R_0603_1608Metric" H 10000 5800 50  0001 C CNN
 F 3 "~" H 10000 5800 50  0001 C CNN
@@
 Text Label 2400 6325 1    50   ~ 0
 SOP2
-Text Label 8100 1925 0    50   ~ 0
-SOP0
-Text Label 8100 1825 0    50   ~ 0
-SOP1
 $Comp
 L Device:R_Small R109
@@
 	0    1    1    0
 $EndComp
-Text Label 2850 925  0    50   ~ 0
+Text Label 2900 975  0    50   ~ 0
 VCC_BRD
 $Comp
@@
 F 2 "Capacitor_SMD:C_0402_1005Metric" H 2575 875 50  0001 C CNN
 F 3 "~" H 2575 875 50  0001 C CNN
-F 4 "TDK" H 2575 875 50  0001 C CNN "MFG Name"
-F 5 "C1005X5R1A104K050BA" H 2575 875 50  0001 C CNN "MFG Part Num"
+F 4 "Murata" H 2575 875 50  0001 C CNN "MFG Name"
+F 5 "GRM155R61A104KA01D" H 2575 875 50  0001 C CNN "MFG Part Num"
 	1    2575 875
 	1    0    0    -1
@@
 L Device:R_Small R132
 U 1 1 5E0B0BBC
-P 950 1750
-F 0 "R132" V 1025 1750 50  0000 C CNN
-F 1 "0" V 875 1750 50  0001 C CNN
-F 2 "Resistor_SMD:R_0402_1005Metric" H 950 1750 50  0001 C CNN
-F 3 "~" H 950 1750 50  0001 C CNN
-F 4 "Panasonic" H 950 1750 50  0001 C CNN "MFG Name"
-F 5 "ERJ-2GE0R00X" H 950 1750 50  0001 C CNN "MFG Part Num"
-	1    950  1750
-	0    1    1    0
-$EndComp
-Text Label 675  1600 3    50   ~ 0
+P 850 1200
+F 0 "R132" V 925 1200 50  0000 C CNN
+F 1 "0" V 775 1200 50  0001 C CNN
+F 2 "Resistor_SMD:R_0402_1005Metric" H 850 1200 50  0001 C CNN
+F 3 "~" H 850 1200 50  0001 C CNN
+F 4 "Panasonic" H 850 1200 50  0001 C CNN "MFG Name"
+F 5 "ERJ-2GE0R00X" H 850 1200 50  0001 C CNN "MFG Part Num"
+	1    850  1200
+	-1   0    0    1
+$EndComp
+Text Label 850  1100 0    50   ~ 0
 SENS_I2C_SCL
 $Comp
 L Device:R_Small R133
 U 1 1 5E11382B
-P 950 1900
-F 0 "R133" V 1025 1900 50  0000 C CNN
-F 1 "0" V 875 1900 50  0001 C CNN
-F 2 "Resistor_SMD:R_0402_1005Metric" H 950 1900 50  0001 C CNN
-F 3 "~" H 950 1900 50  0001 C CNN
-F 4 "Panasonic" H 950 1900 50  0001 C CNN "MFG Name"
-F 5 "ERJ-2GE0R00X" H 950 1900 50  0001 C CNN "MFG Part Num"
-	1    950  1900
-	0    1    1    0
-$EndComp
-Text Label 850  1300 1    50   ~ 0
+P 850 1700
+F 0 "R133" V 925 1700 50  0000 C CNN
+F 1 "0" V 775 1700 50  0001 C CNN
+F 2 "Resistor_SMD:R_0402_1005Metric" H 850 1700 50  0001 C CNN
+F 3 "~" H 850 1700 50  0001 C CNN
+F 4 "Panasonic" H 850 1700 50  0001 C CNN "MFG Name"
+F 5 "ERJ-2GE0R00X" H 850 1700 50  0001 C CNN "MFG Part Num"
+	1    850  1700
+	-1   0    0    1
+$EndComp
+Text Label 850  1800 0    50   ~ 0
 SENS_I2C_SDA
 $Comp
@@
 F 2 "Resistor_SMD:R_0402_1005Metric" H 750 1400 50  0001 C CNN
 F 3 "~" H 750 1400 50  0001 C CNN
-F 4 "Vishay-Dale" H 750 1400 50  0001 C CNN "MFG Name"
-F 5 "CRCW04023K30JNED" H 750 1400 50  0001 C CNN "MFG Part Num"
+F 4 "Panasonic" H 750 1400 50  0001 C CNN "MFG Name"
+F 5 "ERJ-2GE0R00X" H 750 1400 50  0001 C CNN "MFG Part Num"
 	1    750  1400
 	0    1    1    0
@@
 F 2 "Resistor_SMD:R_0402_1005Metric" H 3250 1200 50  0001 C CNN
 F 3 "~" H 3250 1200 50  0001 C CNN
-F 4 "Vishay-Dale" H 3250 1200 50  0001 C CNN "MFG Name"
-F 5 "CRCW04023K30JNED" H 3250 1200 50  0001 C CNN "MFG Part Num"
+F 4 "Panasonic" H 3250 1200 50  0001 C CNN "MFG Name"
+F 5 "ERJ-2GE0R00X" H 3250 1200 50  0001 C CNN "MFG Part Num"
 	1    3250 1200
 	1    0    0    -1
@@
 F 2 "Connector_PinHeader_2.54mm:PinHeader_2x10_P2.54mm_Vertical" H 10025 2400 50  0001 C CNN
 F 3 "~" H 10025 2400 50  0001 C CNN
+F 4 "Wurth" H 10025 2400 50  0001 C CNN "MFG Name"
+F 5 "'61300311121" H 10025 2400 50  0001 C CNN "MFG Part Num"
 	1    10025 2400
 	1    0    0    -1
@@
 	3400 3625 3700 3625
 $Comp
-L wifi-rescue:CC3220MODASF12MONR-2020-05-13_17-39-37 U1
+L wifi-rescue:CC3220MODASF12MONR-2020-05-13_17-39-37 U9
 U 1 1 5F200D4A
 P 4900 4625
-F 0 "U1" H 4900 7013 60  0000 C CNN
+F 0 "U9" H 4900 7013 60  0000 C CNN
 F 1 "CC3220MODASF12MONR" H 4900 6907 60  0000 C CNN
 F 2 "TIMOD_footprints:CC3220MODASF12MONR" H 4900 4565 60  0001 C CNN
 F 3 "" H 4900 4625 60  0000 C CNN
+F 4 "TI" H 4900 4625 50  0001 C CNN "MFG Name"
+F 5 "CC3220MODASF12MONR" H 4900 4625 50  0001 C CNN "MFG Part Num"
 	1    4900 4625
 	1    0    0    -1
@@
 F 2 "Capacitor_SMD:C_0402_1005Metric" H 4875 1400 50  0001 C CNN
 F 3 "~" H 4875 1400 50  0001 C CNN
-F 4 "TDK" H 4875 1400 50  0001 C CNN "MFG Name"
-F 5 "C1005X5R0J475M050BC" H 4875 1400 50  0001 C CNN "MFG Part Num"
+F 4 "Murata" H 4875 1400 50  0001 C CNN "MFG Name"
+F 5 "GRM31CR60J107ME39L" H 4875 1400 50  0001 C CNN "MFG Part Num"
 	1    4875 1400
 	-1   0    0    1
@@
 F 2 "Capacitor_SMD:C_0402_1005Metric" H 5200 1400 50  0001 C CNN
 F 3 "~" H 5200 1400 50  0001 C CNN
-F 4 "TDK" H 5200 1400 50  0001 C CNN "MFG Name"
-F 5 "C1005X5R0J475M050BC" H 5200 1400 50  0001 C CNN "MFG Part Num"
+F 4 "Murata" H 5200 1400 50  0001 C CNN "MFG Name"
+F 5 "GRM31CR60J107ME39L" H 5200 1400 50  0001 C CNN "MFG Part Num"
 	1    5200 1400
 	-1   0    0    1
@@
 F 2 "TMP006_footprints:TMP006AIYZFR" H 4450 1840 60  0001 C CNN
 F 3 "" H 3250 1600 60  0000 C CNN
+F 4 "TI" H 3250 1600 50  0001 C CNN "MFG Name"
+F 5 "TMP006AIYZF" H 3250 1600 50  0001 C CNN "MFG Part Num"
 	1    3250 1600
 	-1   0    0    1
@@
 Connection ~ 3375 2625
 Wire Wire Line
-	675  1600 850  1600
-Wire Wire Line
 	3250 1500 3250 1600
